Commit message: IK options to use Dynamic reachability map (EOXTica IKsolver param) Format conflict: now use eclipse-cpp-google-style

File: tools/dynamic_reachability_map/resources/IndexedCellRobot.urdf (robot description, URDF)
Before this commit: robot IndexedCell, 1 links, 0 joints
Links:
- link base: geometry collision box size=0.1 0.1 0.1; visual box size=0.1 0.1 0.1
