Commit message: [exotica_examples] Moved tests from 'tests' to 'test' directory, moved all test related code/configs to 'test', removed unused tests, upgraded to using rostests/gtest/unittest.

File: examples/exotica_examples/test/resources/Mesh_vs_Mesh_Distance.urdf (robot description, URDF)
Before this commit: robot A_vs_B, 2 links, 1 joints
Links:
- link A: geometry visual mesh filename=package://exotica_examples/test/resources/cube.obj
- link B: geometry visual mesh filename=package://exotica_examples/test/resources/uvsphere.obj

File: examples/exotica_examples/test/resources/Mesh_vs_Mesh_Penetrating.urdf (robot description, URDF)
Before this commit: robot A_vs_B, 2 links, 1 joints
Links:
- link A: geometry visual mesh filename=package://exotica_examples/test/resources/cube.obj
- link B: geometry visual mesh filename=package://exotica_examples/test/resources/uvsphere.obj

File: examples/exotica_examples/test/resources/PrimitiveBox_vs_Mesh_Distance.urdf (robot description, URDF)
Before this commit: robot A_vs_B, 2 links, 1 joints
Links:
- link A: geometry visual box size=2 2 2
- link B: geometry visual mesh filename=package://exotica_examples/test/resources/uvsphere.obj

File: examples/exotica_examples/test/resources/PrimitiveBox_vs_Mesh_Penetrating.urdf (robot description, URDF)
Before this commit: robot A_vs_B, 2 links, 1 joints
Links:
- link B: geometry visual mesh filename=package://exotica_examples/test/resources/uvsphere.obj

File: examples/exotica_examples/test/resources/PrimitiveCylinder_vs_Mesh_Distance.urdf (robot description, URDF)
Before this commit: robot A_vs_B, 2 links, 1 joints
Links:
- link A: geometry visual cylinder length=1 radius=.5
- link B: geometry visual mesh filename=package://exotica_examples/test/resources/uvsphere.obj

File: examples/exotica_examples/test/resources/PrimitiveCylinder_vs_Mesh_Penetrating.urdf (robot description, URDF)
Before this commit: robot A_vs_B, 2 links, 1 joints
Links:
- link A: geometry visual cylinder length=3 radius=.5
- link B: geometry visual mesh filename=package://exotica_examples/test/resources/uvsphere.obj

File: examples/exotica_examples/test/resources/PrimitiveSphere_vs_Mesh_Distance.urdf (robot description, URDF)
Before this commit: robot A_vs_B, 2 links, 1 joints
Links:
- link A: geometry visual sphere radius=1
- link B: geometry visual mesh filename=package://exotica_examples/test/resources/uvsphere.obj

File: examples/exotica_examples/test/resources/PrimitiveSphere_vs_Mesh_Penetrating.urdf (robot description, URDF)
Before this commit: robot A_vs_B, 2 links, 1 joints
Links:
- link A: geometry visual sphere radius=1
- link B: geometry visual mesh filename=package://exotica_examples/test/resources/uvsphere.obj
