Commit message: [exotica_examples] Change test dependency: [val_description] => [exotica_val_description] - Plan to release exotica_val_description

File: examples/exotica_examples/resources/robots/valkyrie_sim.urdf (robot description, URDF)
Before this commit: robot valkyrie, 84 links, 83 joints
Links:
- link hokuyo_link: geometry collision box size=0.08 0.06 0.04238; collision cylinder length=0.047 radius=0.024425
- link leftAnklePitchLink: geometry collision mesh filename=package://exotica_val_description/model/meshes/legs/lj5.dae; visual mesh filename=package://exotica_val_description/model/meshes/legs/lj5.dae
- link leftElbowPitchLink: geometry collision mesh filename=package://exotica_val_description/model/meshes/arms/aj4_lef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; visual mesh filename=package://exotica_val_description/model/meshes/arms/aj4_lef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
- link leftFoot: geometry collision box size=0.27 0.16 0.064; collision sphere radius=0.0
- link leftForearmLink: geometry collision mesh filename=package://exotica_val_description/model/meshes/arms/aj5_lef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; visual mesh filename=package://exotica_val_description/model/meshes/arms/aj5_lef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
- link leftHipPitchLink: geometry collision mesh filename=package://exotica_val_description/model/meshes/legs/lj3_lef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; visual mesh filename=package://exotica_val_description/model/meshes/legs/lj3_lef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
- link leftHipRollLink: geometry collision mesh filename=package://exotica_val_description/model/meshes/legs/lj2_lef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; visual mesh filename=package://exotica_val_description/model/meshes/legs/lj2_lef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
- link leftHipYawLink: geometry collision mesh filename=package://exotica_val_description/model/meshes/legs/lj1_lef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; visual mesh filename=package://exotica_val_description/model/meshes/legs/lj1_lef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
- link leftIndexFingerPitch1Link: geometry collision mesh filename=package://exotica_val_description/model/meshes/fingers/inde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; visual mesh filename=package://exotica_val_description/model/meshes/fingers/inde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
- link leftIndexFingerPitch2Link: geometry collision mesh filename=package://exotica_val_description/model/meshes/fingers/inde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; visual mesh filename=package://exotica_val_description/model/meshes/fingers/inde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
- link leftIndexFingerPitch3Link: geometry collision mesh filename=package://exotica_val_description/model/meshes/fingers/inde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; visual mesh filename=package://exotica_val_description/model/meshes/fingers/inde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
- link leftKneePitchLink: geometry collision mesh filename=package://exotica_val_description/model/meshes/legs/lj4_lef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; visual mesh filename=package://exotica_val_description/model/meshes/legs/lj4_lef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
- link leftMiddleFingerPitch1Link: geometry collision mesh filename=package://exotica_val_description/model/meshes/fingers/midd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; visual mesh filename=package://exotica_val_description/model/meshes/fingers/midd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
- link leftMiddleFingerPitch2Link: geometry collision mesh filename=package://exotica_val_description/model/meshes/fingers/midd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; visual mesh filename=package://exotica_val_description/model/meshes/fingers/midd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
- link leftMiddleFingerPitch3Link: geometry collision mesh filename=package://exotica_val_description/model/meshes/fingers/midd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; visual mesh filename=package://exotica_val_description/model/meshes/fingers/midd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
- link leftPalm: geometry collision mesh filename=package://exotica_val_description/model/meshes/arms/palm_le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; visual mesh filename=package://exotica_val_description/model/meshes/arms/palm_le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
- link leftPinkyPitch1Link: geometry collision mesh filename=package://exotica_val_description/model/meshes/fingers/pink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; visual mesh filename=package://exotica_val_description/model/meshes/fingers/pink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
- link leftPinkyPitch2Link: geometry collision mesh filename=package://exotica_val_description/model/meshes/fingers/pink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; visual mesh filename=package://exotica_val_description/model/meshes/fingers/pink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
- link leftPinkyPitch3Link: geometry collision mesh filename=package://exotica_val_description/model/meshes/fingers/pink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; visual mesh filename=package://exotica_val_description/model/meshes/fingers/pink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
- link leftShoulderPitchLink: geometry collision mesh filename=package://exotica_val_description/model/meshes/arms/aj1_lef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; visual mesh filename=package://exotica_val_description/model/meshes/arms/aj1_lef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
- link leftShoulderRollLink: geometry collision mesh filename=package://exotica_val_description/model/meshes/arms/aj2_lef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; visual mesh filename=package://exotica_val_description/model/meshes/arms/aj2_lef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
- link leftShoulderYawLink: geometry collision mesh filename=package://exotica_val_description/model/meshes/arms/aj3_lef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; visual mesh filename=package://exotica_val_description/model/meshes/arms/aj3_lef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
- link leftThumbPitch1Link: geometry collision mesh filename=package://exotica_val_description/model/meshes/fingers/thum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; visual mesh filename=package://exotica_val_description/model/meshes/fingers/thum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
- link leftThumbPitch2Link: geometry collision mesh filename=package://exotica_val_description/model/meshes/fingers/thum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; visual mesh filename=package://exotica_val_description/model/meshes/fingers/thum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
- link leftThumbPitch3Link: geometry collision mesh filename=package://exotica_val_description/model/meshes/fingers/thum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; visual mesh filename=package://exotica_val_description/model/meshes/fingers/thum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
- link leftThumbRollLink: geometry collision mesh filename=package://exotica_val_description/model/meshes/fingers/thum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; visual mesh filename=package://exotica_val_description/model/meshes/fingers/thum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
- link leftWristRollLink: geometry collision mesh filename=package://exotica_val_description/model/meshes/arms/aj6_lef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; visual mesh filename=package://exotica_val_description/model/meshes/arms/aj6_lef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
- link lowerNeckPitchLink: geometry collision mesh filename=package://exotica_val_description/model/meshes/head/neckj1.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; visual mesh filename=package://exotica_val_description/model/meshes/head/neckj1.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
- link neckYawLink: geometry collision mesh filename=package://exotica_val_description/model/meshes/head/neckj2.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; visual mesh filename=package://exotica_val_description/model/meshes/head/neckj2.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
- link pelvis: geometry collision mesh filename=package://exotica_val_description/model/meshes/pelvis/pelvi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; visual mesh filename=package://exotica_val_description/model/meshes/pelvis/pelvi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
- link rightAnklePitchLink: geometry collision mesh filename=package://exotica_val_description/model/meshes/legs/lj5.dae; visual mesh filename=package://exotica_val_description/model/meshes/legs/lj5.dae
- link rightElbowPitchLink: geometry collision mesh filename=package://exotica_val_description/model/meshes/arms/aj4_rig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; visual mesh filename=package://exotica_val_description/model/meshes/arms/aj4_rig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
- link rightFoot: geometry collision box size=0.27 0.16 0.064; collision sphere radius=0.0
- link rightForearmLink: geometry collision mesh filename=package://exotica_val_description/model/meshes/arms/aj5_rig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; visual mesh filename=package://exotica_val_description/model/meshes/arms/aj5_rig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
- link rightHipPitchLink: geometry collision mesh filename=package://exotica_val_description/model/meshes/legs/lj3_rig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; visual mesh filename=package://exotica_val_description/model/meshes/legs/lj3_rig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
- link rightHipRollLink: geometry collision mesh filename=package://exotica_val_description/model/meshes/legs/lj2_rig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; visual mesh filename=package://exotica_val_description/model/meshes/legs/lj2_rig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
- link rightHipYawLink: geometry collision mesh filename=package://exotica_val_description/model/meshes/legs/lj1_rig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; visual mesh filename=package://exotica_val_description/model/meshes/legs/lj1_rig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
- link rightIndexFingerPitch1Link: geometry collision mesh filename=package://exotica_val_description/model/meshes/fingers/inde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; visual mesh filename=package://exotica_val_description/model/meshes/fingers/inde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
- link rightIndexFingerPitch2Link: geometry collision mesh filename=package://exotica_val_description/model/meshes/fingers/inde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; visual mesh filename=package://exotica_val_description/model/meshes/fingers/inde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
- link rightIndexFingerPitch3Link: geometry collision mesh filename=package://exotica_val_description/model/meshes/fingers/inde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; visual mesh filename=package://exotica_val_description/model/meshes/fingers/inde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
- link rightKneePitchLink: geometry collision mesh filename=package://exotica_val_description/model/meshes/legs/lj4_rig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; visual mesh filename=package://exotica_val_description/model/meshes/legs/lj4_rig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
- link rightMiddleFingerPitch1Link: geometry collision mesh filename=package://exotica_val_description/model/meshes/fingers/midd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; visual mesh filename=package://exotica_val_description/model/meshes/fingers/midd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
- link rightMiddleFingerPitch2Link: geometry collision mesh filename=package://exotica_val_description/model/meshes/fingers/midd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; visual mesh filename=package://exotica_val_description/model/meshes/fingers/midd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
- link rightMiddleFingerPitch3Link: geometry collision mesh filename=package://exotica_val_description/model/meshes/fingers/midd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; visual mesh filename=package://exotica_val_description/model/meshes/fingers/midd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
- link rightPalm: geometry collision mesh filename=package://exotica_val_description/model/meshes/arms/palm_ri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; visual mesh filename=package://exotica_val_description/model/meshes/arms/palm_ri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
- link rightPinkyPitch1Link: geometry collision mesh filename=package://exotica_val_description/model/meshes/fingers/pink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; visual mesh filename=package://exotica_val_description/model/meshes/fingers/pink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
- link rightPinkyPitch2Link: geometry collision mesh filename=package://exotica_val_description/model/meshes/fingers/pink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; visual mesh filename=package://exotica_val_description/model/meshes/fingers/pink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
- link rightPinkyPitch3Link: geometry collision mesh filename=package://exotica_val_description/model/meshes/fingers/pink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; visual mesh filename=package://exotica_val_description/model/meshes/fingers/pink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
- link rightShoulderPitchLink: geometry collision mesh filename=package://exotica_val_description/model/meshes/arms/aj1_rig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; visual mesh filename=package://exotica_val_description/model/meshes/arms/aj1_rig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
- link rightShoulderRollLink: geometry collision mesh filename=package://exotica_val_description/model/meshes/arms/aj2_rig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; visual mesh filename=package://exotica_val_description/model/meshes/arms/aj2_rig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
- link rightShoulderYawLink: geometry collision mesh filename=package://exotica_val_description/model/meshes/arms/aj3_rig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; visual mesh filename=package://exotica_val_description/model/meshes/arms/aj3_rig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
- link rightThumbPitch1Link: geometry collision mesh filename=package://exotica_val_description/model/meshes/fingers/thum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; visual mesh filename=package://exotica_val_description/model/meshes/fingers/thum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
- link rightThumbPitch2Link: geometry collision mesh filename=package://exotica_val_description/model/meshes/fingers/thum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; visual mesh filename=package://exotica_val_description/model/meshes/fingers/thum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
- link rightThumbPitch3Link: geometry collision mesh filename=package://exotica_val_description/model/meshes/fingers/thum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; visual mesh filename=package://exotica_val_description/model/meshes/fingers/thum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
- link rightThumbRollLink: geometry collision mesh filename=package://exotica_val_description/model/meshes/fingers/thum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; visual mesh filename=package://exotica_val_description/model/meshes/fingers/thum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
- link rightWristRollLink: geometry collision mesh filename=package://exotica_val_description/model/meshes/arms/aj6_rig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; visual mesh filename=package://exotica_val_description/model/meshes/arms/aj6_rig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
- link torso: geometry collision mesh filename=package://exotica_val_description/model/meshes/torso/torso.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; visual mesh filename=package://exotica_val_description/model/meshes/torso/torso.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
- link torsoPitchLink: geometry collision mesh filename=package://exotica_val_description/model/meshes/torso/torsop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; visual mesh filename=package://exotica_val_description/model/meshes/torso/torsop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
- link torsoYawLink: geometry collision mesh filename=package://exotica_val_description/model/meshes/torso/torsoy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; visual mesh filename=package://exotica_val_description/model/meshes/torso/torsoy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
- link upperNeckPitchLink: geometry collision mesh filename=package://exotica_val_description/model/meshes/head/head_mu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; visual mesh filename=package://exotica_val_description/model/meshes/head/head_mu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
