Commit message: [exotica_examples] Point to exotica_val_desctiption in the val_simplified.urdf

File: exotica_examples/resources/robots/val_simplified.urdf (robot description, URDF)
Before this commit: robot valkyrie, 84 links, 83 joints
Links:
- link hokuyo_link: geometry collision sphere radius=1e-6; collision sphere radius=1e-6
- link leftAnklePitchLink: geometry collision sphere radius=1e-6; visual mesh filename=package://exotica_val_description/model/meshes/legs/lj5.dae
- link leftElbowPitchLink: geometry collision cylinder length=0.141 radius=0.061; visual mesh filename=package://exotica_val_description/model/meshes/arms/aj4_lef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
- link leftFoot: geometry collision box size=0.27 0.16 0.064; visual mesh filename=package://exotica_val_description/model/meshes/legs/foot.dae
- link leftForearmLink: geometry collision cylinder length=0.22 radius=0.06; visual mesh filename=package://exotica_val_description/model/meshes/arms/aj5_lef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
- link leftHipPitchLink: geometry collision box size=0.22 0.08 0.254; collision box size=0.22 0.22 0.29
- link leftHipRollLink: geometry collision sphere radius=1e-6; visual mesh filename=package://exotica_val_description/model/meshes/legs/lj2_lef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
- link leftHipYawLink: geometry collision sphere radius=0.14; visual mesh filename=package://exotica_val_description/model/meshes/legs/lj1_lef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
- link leftIndexFingerPitch1Link: geometry collision box size=0.015 0.04 0.025; visual mesh filename=package://exotica_val_description/model/meshes/fingers/inde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
- link leftIndexFingerPitch2Link: geometry collision box size=0.015 0.03 0.020; visual mesh filename=package://exotica_val_description/model/meshes/fingers/inde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
- link leftIndexFingerPitch3Link: geometry collision box size=0.015 0.022 0.017; visual mesh filename=package://exotica_val_description/model/meshes/fingers/inde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
- link leftKneePitchLink: geometry collision box size=0.185 0.18 0.38; visual mesh filename=package://exotica_val_description/model/meshes/legs/lj4_lef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
- link leftMiddleFingerPitch1Link: geometry collision box size=0.015 0.04 0.025; visual mesh filename=package://exotica_val_description/model/meshes/fingers/midd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
- link leftMiddleFingerPitch2Link: geometry collision box size=0.015 0.03 0.020; visual mesh filename=package://exotica_val_description/model/meshes/fingers/midd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
- link leftMiddleFingerPitch3Link: geometry collision box size=0.015 0.022 0.017; visual mesh filename=package://exotica_val_description/model/meshes/fingers/midd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
- link leftPalm: geometry collision box size=0.025 0.02 0.12; collision box size=0.03 0.12 0.1
- link leftPinkyPitch1Link: geometry collision box size=0.015 0.04 0.025; visual mesh filename=package://exotica_val_description/model/meshes/fingers/pink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
- link leftPinkyPitch2Link: geometry collision box size=0.015 0.03 0.020; visual mesh filename=package://exotica_val_description/model/meshes/fingers/pink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
- link leftPinkyPitch3Link: geometry collision box size=0.015 0.022 0.017; visual mesh filename=package://exotica_val_description/model/meshes/fingers/pink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
- link leftShoulderPitchLink: geometry collision cylinder length=0.2 radius=0.08; visual mesh filename=package://exotica_val_description/model/meshes/arms/aj1_lef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
- link leftShoulderRollLink: geometry collision cylinder length=0.12 radius=0.075; visual mesh filename=package://exotica_val_description/model/meshes/arms/aj2_lef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
- link leftShoulderYawLink: geometry collision cylinder length=0.20 radius=0.075; visual mesh filename=package://exotica_val_description/model/meshes/arms/aj3_lef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
- link leftThumbPitch1Link: geometry collision box size=0.025 0.015 0.04; visual mesh filename=package://exotica_val_description/model/meshes/fingers/thum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
- link leftThumbPitch2Link: geometry collision box size=0.020 0.015 0.03; visual mesh filename=package://exotica_val_description/model/meshes/fingers/thum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
- link leftThumbPitch3Link: geometry collision box size=0.017 0.015 0.022; visual mesh filename=package://exotica_val_description/model/meshes/fingers/thum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
- link leftThumbRollLink: geometry collision sphere radius=1e-6; visual mesh filename=package://exotica_val_description/model/meshes/fingers/thum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
- link leftWristRollLink: geometry collision sphere radius=1e-6; visual mesh filename=package://exotica_val_description/model/meshes/arms/aj6_lef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
- link lowerNeckPitchLink: geometry collision sphere radius=1e-6; visual mesh filename=package://exotica_val_description/model/meshes/head/neckj1.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
- link neckYawLink: geometry collision sphere radius=1e-6; visual mesh filename=package://exotica_val_description/model/meshes/head/neckj2.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
- link pelvis: geometry collision cylinder length=0.18 radius=0.18; collision sphere radius=0.18
- link rightAnklePitchLink: geometry collision sphere radius=1e-6; visual mesh filename=package://exotica_val_description/model/meshes/legs/lj5.dae
- link rightElbowPitchLink: geometry collision cylinder length=0.141 radius=0.061; visual mesh filename=package://exotica_val_description/model/meshes/arms/aj4_rig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
- link rightFoot: geometry collision box size=0.27 0.16 0.064; visual mesh filename=package://exotica_val_description/model/meshes/legs/foot.dae
- link rightForearmLink: geometry collision cylinder length=0.22 radius=0.06; visual mesh filename=package://exotica_val_description/model/meshes/arms/aj5_rig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
- link rightHipPitchLink: geometry collision box size=0.22 0.08 0.254; collision box size=0.22 0.22 0.29
- link rightHipRollLink: geometry collision sphere radius=1e-6; visual mesh filename=package://exotica_val_description/model/meshes/legs/lj2_rig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
- link rightHipYawLink: geometry collision sphere radius=0.14; visual mesh filename=package://exotica_val_description/model/meshes/legs/lj1_rig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
- link rightIndexFingerPitch1Link: geometry collision box size=0.015 0.04 0.025; visual mesh filename=package://exotica_val_description/model/meshes/fingers/inde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
- link rightIndexFingerPitch2Link: geometry collision box size=0.015 0.03 0.020; visual mesh filename=package://exotica_val_description/model/meshes/fingers/inde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
- link rightIndexFingerPitch3Link: geometry collision box size=0.015 0.022 0.017; visual mesh filename=package://exotica_val_description/model/meshes/fingers/inde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
- link rightKneePitchLink: geometry collision box size=0.185 0.18 0.38; visual mesh filename=package://exotica_val_description/model/meshes/legs/lj4_rig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
- link rightMiddleFingerPitch1Link: geometry collision box size=0.015 0.04 0.025; visual mesh filename=package://exotica_val_description/model/meshes/fingers/midd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
- link rightMiddleFingerPitch2Link: geometry collision box size=0.015 0.03 0.020; visual mesh filename=package://exotica_val_description/model/meshes/fingers/midd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
- link rightMiddleFingerPitch3Link: geometry collision box size=0.015 0.022 0.017; visual mesh filename=package://exotica_val_description/model/meshes/fingers/midd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
- link rightPalm: geometry collision box size=0.03 0.12 0.1; collision cylinder length=0.06 radius=0.05
- link rightPinkyPitch1Link: geometry collision box size=0.015 0.04 0.025; visual mesh filename=package://exotica_val_description/model/meshes/fingers/pink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
- link rightPinkyPitch2Link: geometry collision box size=0.015 0.03 0.020; visual mesh filename=package://exotica_val_description/model/meshes/fingers/pink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
- link rightPinkyPitch3Link: geometry collision box size=0.015 0.022 0.017; visual mesh filename=package://exotica_val_description/model/meshes/fingers/pink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
- link rightShoulderPitchLink: geometry collision cylinder length=0.2 radius=0.08; visual mesh filename=package://exotica_val_description/model/meshes/arms/aj1_rig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
- link rightShoulderRollLink: geometry collision cylinder length=0.12 radius=0.075; visual mesh filename=package://exotica_val_description/model/meshes/arms/aj2_rig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
- link rightShoulderYawLink: geometry collision cylinder length=0.20 radius=0.075; visual mesh filename=package://exotica_val_description/model/meshes/arms/aj3_rig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
- link rightThumbPitch1Link: geometry collision box size=0.025 0.015 0.04; visual mesh filename=package://exotica_val_description/model/meshes/fingers/thum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
- link rightThumbPitch2Link: geometry collision box size=0.020 0.015 0.03; visual mesh filename=package://exotica_val_description/model/meshes/fingers/thum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
- link rightThumbPitch3Link: geometry collision box size=0.017 0.015 0.022; visual mesh filename=package://exotica_val_description/model/meshes/fingers/thum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
- link rightThumbRollLink: geometry collision sphere radius=1e-6; visual mesh filename=package://exotica_val_description/model/meshes/fingers/thum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
- link rightWristRollLink: geometry collision sphere radius=1e-6; visual mesh filename=package://exotica_val_description/model/meshes/arms/aj6_rig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
- link torso: geometry collision box size=0.25 0.36 0.39; collision cylinder length=0.3 radius=0.15
- link torsoPitchLink: geometry collision sphere radius=1e-6; visual mesh filename=package://exotica_val_description/model/meshes/torso/torsop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
- link torsoYawLink: geometry collision sphere radius=1e-6; visual mesh filename=package://exotica_val_description/model/meshes/torso/torsoy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
- link upperNeckPitchLink: geometry collision sphere radius=0.15; visual mesh filename=package://exotica_val_description/model/meshes/head/head_mu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
