Commit message: PR fixes

File: exotica_examples/resources/robots/pendulum.urdf (robot description, URDF)
Before this commit: robot pendulum, 3 links, 2 joints
Links:
- link arm: geometry visual cylinder length=1 radius=0.015
- link base_link: geometry visual cylinder length=0.3 radius=0.04
- link mass: geometry visual box size=0.1 0.1 0.1
