Commit message: [exotica_examples] Remove visuals for head_imu_link, (left/right)_palm, (l/r)_hand_force_torque
These were visual only so in Melodic and older interpreted as collision
links but in Noetic and newer (or MoveIt master in general) only as
visual links.

File: exotica_examples/resources/robots/valkyrie_sim.urdf (robot description, URDF)
Before this commit: robot valkyrie, 84 links, 83 joints
Links:
- link head_imu_link: geometry 
- link l_hand_force_torque: geometry 
- link left_palm: geometry 
- link r_hand_force_torque: geometry 
- link right_palm: geometry 
